Commit message: updating l515 urdf

File: realsense2_description/urdf/_l515.urdf.xacro (robot description, xacro)
@@ -14,5 +14,4 @@
     <!-- The following values are approximate, and the camera node
      publishing TF values with actual calibrated camera extrinsic values -->
-    <xacro:property name="l515_cam_depth_to_infra_offset" value="0.0"/>
     <!-- The following values model the aluminum peripherial case for the
   	L515 camera, with the camera joint represented by the actual
@@ -23,18 +22,12 @@
     <xacro:property name="l515_cam_mount_from_glass_offset" value="0.012"/>
     <!-- Zero depth to glass: see datasheet Revision 002, Fig. 2-2 page 11 -->
-    <xacro:property name="l515_zero_depth_to_glass" value="0.0045"/>
-    <!-- convenience precomputation to avoid clutter-->
-    <xacro:property name="l515_depth_x_offset_from_mount" value="${l515_cam_mount_from_glass_offset-l515_zero_depth_to_glass}"/>
+    <xacro:property name="l515_cam_depth_to_glass" value="0.0045"/>
     <!-- The following offset is relative the the physical D435 camera peripherial
   	camera tripod mount -->
-    <xacro:property name="l515_cam_depth_px" value="${l515_depth_x_offset_from_mount}"/>
-    <xacro:property name="l515_cam_depth_py" value="0.0"/>
     <xacro:property name="l515_cam_center"   value="0.03015"/>
     <xacro:property name="l515_cam_center_to_transmitter_pz"  value="0.001"/>
-    <xacro:property name="l515_cam_transmitter_to_depth_pz"   value="-0.010"/>
-    <xacro:property name="l515_cam_transmitter_to_color_pz"   value="0.014"/>
-    <xacro:property name="l515_cam_depth_pz" value="${l515_cam_center+l515_cam_center_to_transmitter_pz+l515_cam_transmitter_to_depth_pz}"/>
-    <xacro:property name="l515_cam_center_to_depth_pz" value="${l515_cam_center_to_transmitter_pz+l515_cam_transmitter_to_depth_pz}"/>
-    <xacro:property name="abs_mount_from_center"   value="0.020"/>
+    <xacro:property name="l515_cam_transmitter_to_receiver_pz"   value="-0.010"/>
+    <xacro:property name="l515_cam_transmitter_to_rgb_pz"   value="0.014"/>
+    <xacro:property name="l515_cam_mount_from_center"   value="0.020"/>
     <!-- camera body, with origin at bottom screw mount -->
     <joint name="${name}_joint" type="fixed">
@@ -44,13 +37,13 @@
     </joint>
     <link name="${name}_bottom_screw_frame"/>
-    <joint name="${name}_link_joint" type="fixed">
-      <origin xyz="${l515_cam_depth_px} ${l515_cam_depth_py} ${l515_cam_depth_pz}" rpy="0 0 0"/>
+    <joint name="${name}_center_joint" type="fixed">
+      <origin xyz="${l515_cam_mount_from_glass_offset} 0 ${l515_cam_center}" rpy="0 0 0"/>
       <parent link="${name}_bottom_screw_frame"/>
-      <child link="${name}_link" />
+      <child link="${name}_center_frame" />
     </joint>
-    <link name="${name}_link">
+    <link name="${name}_center_frame">
       <visual>
         <!-- the mesh origin is in the middle of the front plate -->
-        <origin xyz="${l515_zero_depth_to_glass} 0 ${-l515_cam_center_to_depth_pz}" rpy="${M_PI/2} 0 ${M_PI/2}"/>
+        <origin xyz="0 0 0" rpy="${M_PI/2} 0 ${M_PI/2}"/>
         <geometry>
 	        <mesh filename="package://realsense2_description/meshes/l515.dae" />
@@ -58,5 +51,5 @@
       </visual>
       <collision>
-        <origin xyz="${-l515_cam_depth_px+l515_cam_mount_from_glass_offset-l515_cam_depth/2} 0 ${-l515_cam_center_to_depth_pz}" rpy="${M_PI/2} 0 ${M_PI/2}"/>
+        <origin xyz="${-l515_cam_depth/2} 0 0" rpy="${M_PI/2} 0 ${M_PI/2}"/>
         <geometry>
           <cylinder radius="${l515_cam_width/2.0}" length="${l515_cam_depth}"/>
@@ -72,5 +65,5 @@
     </link>
     <joint name="${name}_lower_mount_joint" type="fixed">
-      <origin xyz="${l515_cam_mount_from_glass_offset-l515_cam_depth} 0 ${l515_cam_center-abs_mount_from_center}" rpy="0 0 0" />
+      <origin xyz="${l515_cam_mount_from_glass_offset-l515_cam_depth} 0 ${l515_cam_center-l515_cam_mount_from_center}" rpy="0 0 0" />
       <parent link="${name}_bottom_screw_frame" />
       <child link="${name}_lower_mount" />
@@ -78,9 +71,27 @@
     <link name="${name}_lower_mount"/>
     <joint name="${name}_upper_mount_joint" type="fixed">
-      <origin xyz="${l515_cam_mount_from_glass_offset-l515_cam_depth} 0 ${l515_cam_center+abs_mount_from_center}" rpy="0 0 0" />
+      <origin xyz="${l515_cam_mount_from_glass_offset-l515_cam_depth} 0 ${l515_cam_center+l515_cam_mount_from_center}" rpy="0 0 0" />
       <parent link="${name}_bottom_screw_frame" />
       <child link="${name}_upper_mount" />
     </joint>
     <link name="${name}_upper_mount"/>
+    <joint name="${name}_transmitter_joint" type="fixed">
+      <origin xyz="${-l515_cam_depth_to_glass} 0 ${l515_cam_center_to_transmitter_pz}" rpy="0 0 0"/>
+      <parent link="${name}_center_frame"/>
+      <child link="${name}_transmitter_frame" />
+    </joint>
+    <link name="${name}_transmitter_frame"/>
+    <joint name="${name}_receiver_joint" type="fixed">
+      <origin xyz="${l515_cam_depth_to_glass} 0 ${l515_cam_transmitter_to_receiver_pz}" rpy="0 0 0"/>
+      <parent link="${name}_transmitter_frame"/>
+      <child link="${name}_receiver_frame" />
+    </joint>
+    <link name="${name}_receiver_frame"/>
+    <joint name="${name}_rgb_joint" type="fixed">
+      <origin xyz="${l515_cam_depth_to_glass} 0 ${l515_cam_transmitter_to_rgb_pz}" rpy="0 0 0"/>
+      <parent link="${name}_transmitter_frame"/>
+      <child link="${name}_rgb_frame" />
+    </joint>
+    <link name="${name}_rgb_frame"/>
     <!-- Use the nominal extrinsics between camera frames if the calibrated extrinsics aren't being published. e.g. running the device in simulation  -->
     <xacro:if value="${use_nominal_extrinsics}">
@@ -88,5 +99,5 @@
       <joint name="${name}_depth_joint" type="fixed">
         <origin xyz="0 0 0" rpy="0 0 0"/>
-        <parent link="${name}_link"/>
+        <parent link="${name}_transmitter_frame"/>
         <child link="${name}_depth_frame" />
       </joint>
@@ -98,8 +109,8 @@
       </joint>
       <link name="${name}_depth_optical_frame"/>
-      <!-- camera left IR joints and links -->
+      <!-- camera IR joints and links -->
       <joint name="${name}_infra_joint" type="fixed">
-        <origin xyz="0 ${l515_cam_depth_to_infra_offset} 0" rpy="0 0 0" />
-        <parent link="${name}_link" />
+        <origin xyz="0 0 0" rpy="0 0 0" />
+        <parent link="${name}_receiver_frame" />
         <child link="${name}_infra_frame" />
       </joint>
@@ -113,6 +124,6 @@
       <!-- camera color joints and links -->
       <joint name="${name}_color_joint" type="fixed">
-        <origin xyz="0 0 ${-l515_cam_transmitter_to_depth_pz+l515_cam_transmitter_to_color_pz}" rpy="0 0 0" />
-        <parent link="${name}_link" />
+        <origin xyz="0 0 0" rpy="0 0 0" />
+        <parent link="${name}_rgb_frame" />
         <child link="${name}_color_frame" />
       </joint>

Commit message: adding depth rotation offset

File: realsense2_description/urdf/_l515.urdf.xacro (robot description, xacro)
@@ -22,5 +22,5 @@
     <xacro:property name="l515_cam_mount_from_glass_offset" value="0.012"/>
     <!-- Zero depth to glass: see datasheet Revision 002, Fig. 2-2 page 11 -->
-    <xacro:property name="l515_cam_depth_to_glass" value="0.0045"/>
+    <xacro:property name="l515_cam_depth_to_glass" value="0.0044533"/>
     <!-- The following offset is relative the the physical D435 camera peripherial
   	camera tripod mount -->
@@ -28,5 +28,5 @@
     <xacro:property name="l515_cam_center_to_transmitter_pz"  value="0.001"/>
     <xacro:property name="l515_cam_transmitter_to_receiver_pz"   value="-0.010"/>
-    <xacro:property name="l515_cam_transmitter_to_rgb_pz"   value="0.014"/>
+    <xacro:property name="l515_cam_transmitter_to_rgb_pz"   value="0.014182"/>
     <xacro:property name="l515_cam_mount_from_center"   value="0.020"/>
     <!-- camera body, with origin at bottom screw mount -->
@@ -98,5 +98,5 @@
       <!-- camera depth joints and links -->
       <joint name="${name}_depth_joint" type="fixed">
-        <origin xyz="0 0 0" rpy="0 0 0"/>
+        <origin xyz="0 0 0" rpy="0 0 0"/> <!-- -0.016 0.028 0.016 -->
         <parent link="${name}_transmitter_frame"/>
         <child link="${name}_depth_frame" />

Commit message: fixing depth rotation offset

File: realsense2_description/urdf/_l515.urdf.xacro (robot description, xacro)
@@ -98,5 +98,5 @@
       <!-- camera depth joints and links -->
       <joint name="${name}_depth_joint" type="fixed">
-        <origin xyz="0 0 0" rpy="0 0 0"/> <!-- -0.016 0.028 0.016 -->
+        <origin xyz="0 0 0" rpy="-0.016 0.0 0.016"/>
         <parent link="${name}_transmitter_frame"/>
         <child link="${name}_depth_frame" />
@@ -124,5 +124,5 @@
       <!-- camera color joints and links -->
       <joint name="${name}_color_joint" type="fixed">
-        <origin xyz="0 0 0" rpy="0 0 0" />
+        <origin xyz="0 0 0" rpy="0 -0.028 0" />
         <parent link="${name}_rgb_frame" />
         <child link="${name}_color_frame" />

Commit message: increasing realsense collision box size

File: realsense2_description/urdf/_l515.urdf.xacro (robot description, xacro)
@@ -53,5 +53,5 @@
         <origin xyz="${-l515_cam_depth/2} 0 0" rpy="${M_PI/2} 0 ${M_PI/2}"/>
         <geometry>
-          <cylinder radius="${l515_cam_width/2.0}" length="${l515_cam_depth}"/>
+          <cylinder radius="${l515_cam_width}" length="${l515_cam_depth}"/>
         </geometry>
       </collision>

Commit message: adding in imu frames

File: realsense2_description/urdf/_l515.urdf.xacro (robot description, xacro)
@@ -30,4 +30,12 @@
     <xacro:property name="l515_cam_transmitter_to_rgb_pz"   value="0.014182"/>
     <xacro:property name="l515_cam_mount_from_center"   value="0.020"/>
+    <!-- IMU position (p) and rotation (r) offsets from the camera color frame -->
+    <!-- These values are approximate and depend on the actual calibrated camera extrinsic values -->
+    <xacro:property name="l515_cam_color_to_imu_px" value="-0.00410137791186571"/>
+    <xacro:property name="l515_cam_color_to_imu_py" value="-0.0129784867167473"/>
+    <xacro:property name="l515_cam_color_to_imu_pz" value="0.00256138201802969"/>
+    <xacro:property name="l515_cam_color_to_imu_rx" value="-0.006161012"/>
+    <xacro:property name="l515_cam_color_to_imu_ry" value="0.020193459"/>
+    <xacro:property name="l515_cam_color_to_imu_rz" value="0.016301375"/>
     <!-- camera body, with origin at bottom screw mount -->
     <joint name="${name}_joint" type="fixed">
@@ -135,4 +143,41 @@
       </joint>
       <link name="${name}_color_optical_frame"/>
+      <!-- camera IMU joints and links -->
+      <link name="${name}_gyro_frame" />
+      <link name="${name}_gyro_optical_frame" />
+      <link name="${name}_accel_frame" />
+      <link name="${name}_accel_optical_frame" />
+      <link name="${name}_imu_frame" />
+      <link name="${name}_imu_optical_frame" />
+      <joint name="${name}_gyro_joint" type="fixed">
+        <origin xyz = "${l515_cam_color_to_imu_px} ${l515_cam_color_to_imu_py} ${l515_cam_color_to_imu_pz}" rpy = "${l515_cam_color_to_imu_rx} ${l515_cam_color_to_imu_ry} ${l515_cam_color_to_imu_rz}" />
+        <parent link="${name}_color_frame" />
+        <child link="${name}_gyro_frame" />
+      </joint>
+      <joint name="${name}_gyro_optical_joint" type="fixed">
+        <origin xyz = "0 0 0" rpy = "${-M_PI/2} 0 ${-M_PI/2}" />
+        <parent link="${name}_gyro_frame" />
+        <child link="${name}_gyro_optical_frame" />
+      </joint>
+      <joint name="${name}_accel_joint" type="fixed">
+        <origin xyz = "${l515_cam_color_to_imu_px} ${l515_cam_color_to_imu_py} ${l515_cam_color_to_imu_pz}" rpy = "${l515_cam_color_to_imu_rx} ${l515_cam_color_to_imu_ry} ${l515_cam_color_to_imu_rz}" />
+        <parent link="${name}_color_frame" />
+        <child link="${name}_accel_frame" />
+      </joint>
+      <joint name="${name}_accel_optical_joint" type="fixed">
+        <origin xyz = "0 0 0" rpy = "${-M_PI/2} 0 ${-M_PI/2}" />
+        <parent link="${name}_accel_frame" />
+        <child link="${name}_accel_optical_frame" />
+      </joint>
+      <joint name="${name}_imu_joint" type="fixed">
+        <origin xyz = "${l515_cam_color_to_imu_px} ${l515_cam_color_to_imu_py} ${l515_cam_color_to_imu_pz}" rpy = "${l515_cam_color_to_imu_rx} ${l515_cam_color_to_imu_ry} ${l515_cam_color_to_imu_rz}" />
+        <parent link="${name}_color_frame" />
+        <child link="${name}_imu_frame" />
+      </joint>
+      <joint name="${name}_imu_optical_joint" type="fixed">
+        <origin xyz = "0 0 0" rpy = "${-M_PI/2} 0 ${-M_PI/2}" />
+        <parent link="${name}_imu_frame" />
+        <child link="${name}_imu_optical_frame" />
+      </joint>
     </xacro:if>
     <xacro:if value="${add_plug}">

Commit message: updating l515 urdf to use published extrinsics

File: realsense2_description/urdf/_l515.urdf.xacro (robot description, xacro)
@@ -7,8 +7,5 @@
 -->
 <robot name="sensor_l515" xmlns:xacro="http://ros.org/wiki/xacro">
-  <!-- Includes -->
-  <xacro:include filename="$(find realsense2_description)/urdf/_materials.urdf.xacro" />
-  <xacro:include filename="$(find realsense2_description)/urdf/_usb_plug.urdf.xacro" /> <!-- this specific plug does not apply to L515 -->
-  <xacro:macro name="sensor_l515" params="parent *origin name:=camera use_nominal_extrinsics:=false add_plug:=false use_mesh:=true">
+  <xacro:macro name="sensor_l515" params="parent *origin name:=camera use_nominal_extrinsics:=false">
     <xacro:property name="M_PI" value="3.1415926535897931" />
     <!-- The following values are approximate, and the camera node
@@ -104,4 +101,10 @@
     </joint>
     <link name="${name}_receiver_frame"/>
+    <joint name="${name}_link_joint" type="fixed">
+      <origin xyz="0 0 0" rpy="0 0 0"/>
+      <parent link="${name}_receiver_frame"/>
+      <child link="${name}_link" />
+    </joint>
+    <link name="${name}_link"/>
     <joint name="${name}_rgb_joint" type="fixed">
       <origin xyz="${l515_cam_depth_to_glass} 0 ${l515_cam_transmitter_to_rgb_pz}" rpy="0 0 0"/>
@@ -110,5 +113,5 @@
     </joint>
     <link name="${name}_rgb_frame"/>
-    <!-- Use the nominal extrinsics between camera frames if the calibrated extrinsics aren't being published. e.g. running the device in simulation  -->
+    <!-- Use the nominal extrinsics between camera frames if the calibrated extrinsics aren't being published -->
     <xacro:if value="${use_nominal_extrinsics}">
       <!-- camera depth joints and links -->
@@ -189,9 +192,4 @@
       </joint>
     </xacro:if>
-    <xacro:if value="${add_plug}">
-      <xacro:usb_plug parent="${name}_bottom_screw_frame" name="${name}_usb_plug">
-        <origin xyz="${l515_cam_mount_from_glass_offset-0.0148} -0.018 0.018" rpy="${M_PI/4} 0 0 "/>
-      </xacro:usb_plug>
-    </xacro:if>
   </xacro:macro>
 </robot>

Commit message: updating imu transforms

File: realsense2_description/urdf/_l515.urdf.xacro (robot description, xacro)
@@ -22,5 +22,5 @@
     <xacro:property name="l515_cam_mount_from_glass_offset" value="0.012"/>
     <!-- Zero depth to glass: see datasheet Revision 002, Fig. 2-2 page 11 -->
-    <xacro:property name="l515_cam_depth_to_glass" value="0.0044533"/>
+    <xacro:property name="l515_cam_depth_to_glass" value="0.0045"/>
     <!-- The following offset is relative the the physical D435 camera peripherial
   	camera tripod mount -->
@@ -28,14 +28,8 @@
     <xacro:property name="l515_cam_center_to_transmitter_pz"  value="0.001"/>
     <xacro:property name="l515_cam_transmitter_to_receiver_pz"   value="-0.010"/>
-    <xacro:property name="l515_cam_transmitter_to_rgb_pz"   value="0.014182"/>
+    <xacro:property name="l515_cam_transmitter_to_rgb_pz"   value="0.014"/>
     <xacro:property name="l515_cam_mount_from_center"   value="0.020"/>
-    <!-- IMU position (p) and rotation (r) offsets from the camera color frame -->
-    <!-- These values are approximate and depend on the actual calibrated camera extrinsic values -->
-    <xacro:property name="l515_cam_color_to_imu_px" value="-0.00410137791186571"/>
-    <xacro:property name="l515_cam_color_to_imu_py" value="-0.0129784867167473"/>
-    <xacro:property name="l515_cam_color_to_imu_pz" value="0.00256138201802969"/>
-    <xacro:property name="l515_cam_color_to_imu_rx" value="-0.006161012"/>
-    <xacro:property name="l515_cam_color_to_imu_ry" value="0.020193459"/>
-    <xacro:property name="l515_cam_color_to_imu_rz" value="0.016301375"/>
+    <xacro:property name="l515_cam_transmitter_to_imu_py" value="-0.01245"/>
+    <xacro:property name="l515_cam_transmitter_to_imu_pz" value="0.0105"/>
     <!-- camera body, with origin at bottom screw mount -->
     <joint name="${name}_joint" type="fixed">
@@ -102,4 +96,10 @@
     </joint>
     <link name="${name}_rgb_frame"/>
+    <joint name="${name}_imu_joint" type="fixed">
+      <origin xyz = "0 ${l515_cam_transmitter_to_imu_py} ${l515_cam_transmitter_to_imu_pz}" rpy = "0 0 0" />
+      <parent link="${name}_transmitter_frame" />
+      <child link="${name}_imu_frame" />
+    </joint>
+    <link name="${name}_imu_frame" />
     <!-- Use the nominal extrinsics between camera frames if the calibrated extrinsics aren't being published. e.g. running the device in simulation  -->
     <xacro:if value="${use_nominal_extrinsics}">
@@ -143,36 +143,4 @@
       </joint>
       <link name="${name}_color_optical_frame"/>
-      <!-- camera IMU joints and links -->
-      <link name="${name}_gyro_frame" />
-      <link name="${name}_gyro_optical_frame" />
-      <link name="${name}_accel_frame" />
-      <link name="${name}_accel_optical_frame" />
-      <link name="${name}_imu_frame" />
-      <link name="${name}_imu_optical_frame" />
-      <joint name="${name}_gyro_joint" type="fixed">
-        <origin xyz = "${l515_cam_color_to_imu_px} ${l515_cam_color_to_imu_py} ${l515_cam_color_to_imu_pz}" rpy = "${l515_cam_color_to_imu_rx} ${l515_cam_color_to_imu_ry} ${l515_cam_color_to_imu_rz}" />
-        <parent link="${name}_color_frame" />
-        <child link="${name}_gyro_frame" />
-      </joint>
-      <joint name="${name}_gyro_optical_joint" type="fixed">
-        <origin xyz = "0 0 0" rpy = "${-M_PI/2} 0 ${-M_PI/2}" />
-        <parent link="${name}_gyro_frame" />
-        <child link="${name}_gyro_optical_frame" />
-      </joint>
-      <joint name="${name}_accel_joint" type="fixed">
-        <origin xyz = "${l515_cam_color_to_imu_px} ${l515_cam_color_to_imu_py} ${l515_cam_color_to_imu_pz}" rpy = "${l515_cam_color_to_imu_rx} ${l515_cam_color_to_imu_ry} ${l515_cam_color_to_imu_rz}" />
-        <parent link="${name}_color_frame" />
-        <child link="${name}_accel_frame" />
-      </joint>
-      <joint name="${name}_accel_optical_joint" type="fixed">
-        <origin xyz = "0 0 0" rpy = "${-M_PI/2} 0 ${-M_PI/2}" />
-        <parent link="${name}_accel_frame" />
-        <child link="${name}_accel_optical_frame" />
-      </joint>
-      <joint name="${name}_imu_joint" type="fixed">
-        <origin xyz = "${l515_cam_color_to_imu_px} ${l515_cam_color_to_imu_py} ${l515_cam_color_to_imu_pz}" rpy = "${l515_cam_color_to_imu_rx} ${l515_cam_color_to_imu_ry} ${l515_cam_color_to_imu_rz}" />
-        <parent link="${name}_color_frame" />
-        <child link="${name}_imu_frame" />
-      </joint>
       <joint name="${name}_imu_optical_joint" type="fixed">
         <origin xyz = "0 0 0" rpy = "${-M_PI/2} 0 ${-M_PI/2}" />
@@ -180,4 +148,5 @@
         <child link="${name}_imu_optical_frame" />
       </joint>
+      <link name="${name}_imu_optical_frame" />
     </xacro:if>
     <xacro:if value="${add_plug}">

Commit message: updating imu transforms

File: realsense2_description/urdf/_l515.urdf.xacro (robot description, xacro)
@@ -31,5 +31,5 @@
     <xacro:property name="l515_cam_mount_from_center"   value="0.020"/>
     <xacro:property name="l515_cam_transmitter_to_imu_py" value="-0.01245"/>
-    <xacro:property name="l515_cam_transmitter_to_imu_pz" value="0.0105"/>
+    <xacro:property name="l515_cam_transmitter_to_imu_pz" value="0.01151"/>
     <!-- camera body, with origin at bottom screw mount -->
     <joint name="${name}_joint" type="fixed">

Commit message: updating l515 xacro

File: realsense2_description/urdf/_l515.urdf.xacro (robot description, xacro)
@@ -22,19 +22,11 @@
     <!-- The following offset is relative the the physical L515 camera peripherial
   	camera tripod mount -->
-    <xacro:property name="l515_cam_center"   value="0.03015"/>
-    <xacro:property name="l515_cam_center_to_transmitter_pz"  value="0.001"/>
-    <xacro:property name="l515_cam_transmitter_to_receiver_pz"   value="-0.010"/>
-    <xacro:property name="l515_cam_transmitter_to_rgb_pz"   value="0.014"/>
-    <xacro:property name="l515_cam_mount_from_center"   value="0.020"/>
+    <xacro:property name="l515_cam_center" value="0.03015"/>
+    <xacro:property name="l515_cam_center_to_transmitter_pz" value="0.001"/>
+    <xacro:property name="l515_cam_transmitter_to_receiver_pz" value="-0.010"/>
+    <xacro:property name="l515_cam_transmitter_to_rgb_pz" value="0.014"/>
+    <xacro:property name="l515_cam_mount_from_center" value="0.020"/>
     <xacro:property name="l515_cam_transmitter_to_imu_py" value="-0.01245"/>
     <xacro:property name="l515_cam_transmitter_to_imu_pz" value="0.01151"/>
-    <!-- IMU position (p) and rotation (r) offsets from the camera color frame -->
-    <!-- These values are approximate and depend on the actual calibrated camera extrinsic values -->
-    <xacro:property name="l515_cam_color_to_imu_px" value="-0.00410137791186571"/>
-    <xacro:property name="l515_cam_color_to_imu_py" value="-0.0129784867167473"/>
-    <xacro:property name="l515_cam_color_to_imu_pz" value="0.00256138201802969"/>
-    <xacro:property name="l515_cam_color_to_imu_rx" value="-0.006161012"/>
-    <xacro:property name="l515_cam_color_to_imu_ry" value="0.020193459"/>
-    <xacro:property name="l515_cam_color_to_imu_rz" value="0.016301375"/>
     <!-- camera body, with origin at bottom screw mount -->
     <joint name="${name}_joint" type="fixed">
@@ -63,11 +55,4 @@
         </geometry>
       </collision>
-      <inertial>
-        <!-- The following are not reliable values, and should not be used for modeling -->
-        <!-- calculated assuming full cylinder as described here: https://en.wikipedia.org/wiki/List_of_moments_of_inertia -->
-        <mass value="0.095" />
-        <origin xyz="0 0 0" />
-        <inertia ixx="0.000044" ixy="0.0" ixz="0.0" iyy="0.000027" iyz="0.0" izz="0.000027" />
-      </inertial>
     </link>
     <joint name="${name}_lower_mount_joint" type="fixed">
