Commit message: updating l515 frames

File: realsense2_description/urdf/_l515.urdf.xacro (robot description, xacro)
@@ -80,10 +80,4 @@
     </joint>
     <link name="${name}_receiver_frame"/>
-    <joint name="${name}_link_joint" type="fixed">
-      <origin xyz="0 0 0" rpy="0 0 0"/>
-      <parent link="${name}_receiver_frame"/>
-      <child link="${name}_link" />
-    </joint>
-    <link name="${name}_link"/>
     <joint name="${name}_rgb_joint" type="fixed">
       <origin xyz="${l515_cam_depth_to_glass} 0 ${l515_cam_transmitter_to_rgb_pz}" rpy="0 0 0"/>

Commit message: updating l515 urdf

File: realsense2_description/urdf/_l515.urdf.xacro (robot description, xacro)
@@ -19,5 +19,5 @@
     <xacro:property name="l515_cam_mount_from_glass_offset" value="0.012"/>
     <!-- Zero depth to glass: see datasheet Revision 002, Fig. 2-2 page 11 -->
-    <xacro:property name="l515_cam_depth_to_glass" value="0.0045"/>
+    <xacro:property name="l515_cam_depth_to_glass" value="0.004"/>
     <!-- The following offset is relative the the physical L515 camera peripherial
   	camera tripod mount -->
@@ -27,6 +27,7 @@
     <xacro:property name="l515_cam_transmitter_to_rgb_pz" value="0.014"/>
     <xacro:property name="l515_cam_mount_from_center" value="0.020"/>
-    <xacro:property name="l515_cam_transmitter_to_imu_py" value="-0.01245"/>
-    <xacro:property name="l515_cam_transmitter_to_imu_pz" value="0.01151"/>
+    <xacro:property name="l515_cam_transmitter_to_imu_px" value="-0.001"/>
+    <xacro:property name="l515_cam_transmitter_to_imu_py" value="-0.012"/>
+    <xacro:property name="l515_cam_transmitter_to_imu_pz" value="0.016"/>
     <!-- camera body, with origin at bottom screw mount -->
     <joint name="${name}_joint" type="fixed">
@@ -87,5 +88,5 @@
     <link name="${name}_rgb_frame"/>
     <joint name="${name}_imu_joint" type="fixed">
-      <origin xyz = "0 ${l515_cam_transmitter_to_imu_py} ${l515_cam_transmitter_to_imu_pz}" rpy = "0 0 0" />
+      <origin xyz = "${l515_cam_transmitter_to_imu_px} ${l515_cam_transmitter_to_imu_py} ${l515_cam_transmitter_to_imu_pz}" rpy = "0 0 0" />
       <parent link="${name}_transmitter_frame" />
       <child link="${name}_imu_frame" />
